File: PCB/Satellite.kicad_pcb (KiCad board)
At the start: 2 copper layers, 300 x 80 mm, 124 parts, among them SW1 SW_Push, SW10 SW_Push, SW11 SW_Push, SW12 SW_Push, SW13 SW_Push, SW14 SW_Push, SW15 SW_Push, SW16 SW_Push, SW17 SW_Push, SW18 SW_Push, SW19 SW_Push, SW2 SW_Push, SW20 SW_Push, SW21 SW_Push, SW22 SW_Push, SW23 SW_Push, SW24 SW_Push, SW25 SW_Push, SW26 SW_Push, SW27 SW_Push, SW28 SW_Push, SW29 SW_Push, SW3 SW_Push, SW30 SW_Push, SW31 SW_Push, SW32 SW_Push, SW33 SW_Push, SW34 SW_Push, SW35 SW_Push, SW36 SW_Push, SW37 SW_Push, SW38 SW_Push, SW39 SW_Push, SW4 SW_Push, SW40 SW_Push, SW41 SW_Push, SW42 SW_Push, SW43 SW_Push, SW44 SW_Push, SW45 SW_Push, SW46 SW_Push, SW47 SW_Push, SW48 SW_Push, SW5 SW_Push, SW6 SW_Push, SW7 SW_Push, SW8 SW_Push, SW9 SW_Push, Y1 16Mhz

Commit message: Hybrid Socket upgrade
Parts:
- SW1, SW10, SW11, SW12, SW13, SW14, SW15, SW16, SW17, SW18, SW19, SW2, SW20, SW21, SW22, SW23, SW24, SW25, SW26, SW27, SW28, SW29, SW3, SW30, SW31, SW32, SW33, SW34, SW35, SW36, SW37, SW38, SW39, SW4, SW40, SW41, SW42, SW43, SW44, SW45, SW46, SW47, SW48, SW5, SW6, SW7, SW8, SW9: footprint Button_Switch_Keyboard:SW_Cherry_MX_1.00u_PCB -> MX_Alps_Hybrid:MX-1U-NoLED
- U1: renamed from ATmega 328P
- moved SW18 5.68 mm to (129.6, 56.3)
- moved SW22 5.68 mm to (274.5, 56.3)
- moved SW23 5.68 mm to (293.5, 56.3)
- moved SW10 5.68 mm to (274.5, 37.3)
- moved SW11 5.68 mm to (293.5, 37.3)
- moved SW15 5.68 mm to (72.5, 56.3)
- moved SW16 5.68 mm to (91.5, 56.3)
- moved SW17 5.68 mm to (110.6, 56.3)
- moved SW30 5.68 mm to (129.6, 75.4)
- moved SW34 5.68 mm to (274.5, 75.4)
- moved SW35 5.68 mm to (293.5, 75.4)
- moved SW42 5.68 mm to (129.6, 94.4)
- moved SW46 5.68 mm to (274.5, 94.4)
- moved SW47 5.68 mm to (293.5, 94.4)
- moved SW6 5.68 mm to (129.6, 37.3)
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- renumbered ISP to J2, I2C to J3, RESET to SW49, BOOT to SW50
Connections:
- J2 pad 1: /COL5 -> /COL0
- J2 pad 3: /COL4 -> /COL1
- SW1 pad 1: /COL6 -> Net-(D1-Pad2)
- SW1 pad 2: Net-(D1-Pad2) -> /COL6
- SW10 pad 1: /COL3 -> Net-(D10-Pad2)
- SW10 pad 2: Net-(D10-Pad2) -> /COL3
- SW11 pad 1: /COL4 -> Net-(D11-Pad2)
- SW11 pad 2: Net-(D11-Pad2) -> /COL4
- SW12 pad 1: /COL5 -> Net-(D12-Pad2)
- SW12 pad 2: Net-(D12-Pad2) -> /COL5
- SW13 pad 1: /COL6 -> Net-(D13-Pad2)
- SW13 pad 2: Net-(D13-Pad2) -> /COL6
- SW14 pad 1: /COL7 -> Net-(D14-Pad2)
- SW14 pad 2: Net-(D14-Pad2) -> /COL7
- SW15 pad 1: /COL8 -> Net-(D15-Pad2)
- SW15 pad 2: Net-(D15-Pad2) -> /COL8
- SW16 pad 1: /COL9 -> Net-(D16-Pad2)
- SW16 pad 2: Net-(D16-Pad2) -> /COL9
- SW17 pad 1: /COL10 -> Net-(D17-Pad2)
- SW17 pad 2: Net-(D17-Pad2) -> /COL10
- SW18 pad 1: /COL11 -> Net-(D18-Pad2)
- SW18 pad 2: Net-(D18-Pad2) -> /COL11
- SW19 pad 1: /COL0 -> Net-(D19-Pad2)
- SW19 pad 2: Net-(D19-Pad2) -> /COL0
- SW2 pad 1: /COL7 -> Net-(D2-Pad2)
- SW2 pad 2: Net-(D2-Pad2) -> /COL7
- SW20 pad 1: /COL1 -> Net-(D20-Pad2)
- SW20 pad 2: Net-(D20-Pad2) -> /COL1
- SW21 pad 1: /COL2 -> Net-(D21-Pad2)
- SW21 pad 2: Net-(D21-Pad2) -> /COL2
- SW22 pad 1: /COL3 -> Net-(D22-Pad2)
- SW22 pad 2: Net-(D22-Pad2) -> /COL3
- SW23 pad 1: /COL4 -> Net-(D23-Pad2)
- SW23 pad 2: Net-(D23-Pad2) -> /COL4
- SW24 pad 1: /COL5 -> Net-(D24-Pad2)
- SW24 pad 2: Net-(D24-Pad2) -> /COL5
- SW25 pad 1: /COL6 -> Net-(D25-Pad2)
- SW25 pad 2: Net-(D25-Pad2) -> /COL6
- SW26 pad 1: /COL7 -> Net-(D26-Pad2)
- SW26 pad 2: Net-(D26-Pad2) -> /COL7
- SW27 pad 1: /COL8 -> Net-(D27-Pad2)
- SW27 pad 2: Net-(D27-Pad2) -> /COL8
- SW28 pad 1: /COL9 -> Net-(D28-Pad2)
- SW28 pad 2: Net-(D28-Pad2) -> /COL9
- SW29 pad 1: /COL10 -> Net-(D29-Pad2)
- SW29 pad 2: Net-(D29-Pad2) -> /COL10
- SW3 pad 1: /COL8 -> Net-(D3-Pad2)
- SW3 pad 2: Net-(D3-Pad2) -> /COL8
- SW30 pad 1: /COL11 -> Net-(D30-Pad2)
- SW30 pad 2: Net-(D30-Pad2) -> /COL11
- SW31 pad 1: /COL0 -> Net-(D31-Pad2)
- SW31 pad 2: Net-(D31-Pad2) -> /COL0
- SW32 pad 1: /COL1 -> Net-(D32-Pad2)
- SW32 pad 2: Net-(D32-Pad2) -> /COL1
- SW33 pad 1: /COL2 -> Net-(D33-Pad2)
- SW33 pad 2: Net-(D33-Pad2) -> /COL2
- SW34 pad 1: /COL3 -> Net-(D34-Pad2)
- SW34 pad 2: Net-(D34-Pad2) -> /COL3
- SW35 pad 1: /COL4 -> Net-(D35-Pad2)
- SW35 pad 2: Net-(D35-Pad2) -> /COL4
- SW36 pad 1: /COL5 -> Net-(D36-Pad2)
- SW36 pad 2: Net-(D36-Pad2) -> /COL5
- SW37 pad 1: /COL6 -> Net-(D37-Pad2)
- SW37 pad 2: Net-(D37-Pad2) -> /COL6
- SW38 pad 1: /COL7 -> Net-(D38-Pad2)
- SW38 pad 2: Net-(D38-Pad2) -> /COL7
- SW39 pad 1: /COL8 -> Net-(D39-Pad2)
- SW39 pad 2: Net-(D39-Pad2) -> /COL8
- SW4 pad 1: /COL9 -> Net-(D4-Pad2)
- SW4 pad 2: Net-(D4-Pad2) -> /COL9
- SW40 pad 1: /COL9 -> Net-(D40-Pad2)
- SW40 pad 2: Net-(D40-Pad2) -> /COL9
- SW41 pad 1: /COL10 -> Net-(D41-Pad2)
- SW41 pad 2: Net-(D41-Pad2) -> /COL10
- SW42 pad 1: /COL11 -> Net-(D42-Pad2)
- SW42 pad 2: Net-(D42-Pad2) -> /COL11
- SW43 pad 1: /COL0 -> Net-(D43-Pad2)
- SW43 pad 2: Net-(D43-Pad2) -> /COL0
- SW44 pad 1: /COL1 -> Net-(D44-Pad2)
- SW44 pad 2: Net-(D44-Pad2) -> /COL1
- SW45 pad 1: /COL2 -> Net-(D45-Pad2)
- SW45 pad 2: Net-(D45-Pad2) -> /COL2
- SW46 pad 1: /COL3 -> Net-(D46-Pad2)
- SW46 pad 2: Net-(D46-Pad2) -> /COL3
- SW47 pad 1: /COL4 -> Net-(D47-Pad2)
- SW47 pad 2: Net-(D47-Pad2) -> /COL4
- SW48 pad 1: /COL5 -> Net-(D48-Pad2)
- SW48 pad 2: Net-(D48-Pad2) -> /COL5
- SW49 pad 1: /RESET -> GND
- SW49 pad 2: GND -> /RESET
- SW5 pad 1: /COL10 -> Net-(D5-Pad2)
- SW5 pad 2: Net-(D5-Pad2) -> /COL10
- SW50 pad 1: /COL8 -> GND
- SW50 pad 2: GND -> /COL8
- SW6 pad 1: /COL11 -> Net-(D6-Pad2)
- SW6 pad 2: Net-(D6-Pad2) -> /COL11
- SW7 pad 1: /COL0 -> Net-(D7-Pad2)
- SW7 pad 2: Net-(D7-Pad2) -> /COL0
- SW8 pad 1: /COL1 -> Net-(D8-Pad2)
- SW8 pad 2: Net-(D8-Pad2) -> /COL1
- SW9 pad 1: /COL2 -> Net-(D9-Pad2)
- SW9 pad 2: Net-(D9-Pad2) -> /COL2
Routing:
- net /COL8: track 266.9 -> 272.3 mm
- net GND: track 170.5 -> 173.7 mm
- net /RESET: track 121.4 -> 123.0 mm

Commit message: PCB minor
Parts:
- I2C: renamed from J3; footprint Connector_Wire:SolderWirePad_1x04_P3.175mm_Drill0.8mm -> Connector_PinHeader_2.00mm:PinHeader_1x04_P2.00mm_Vertical
- moved I2C 1.52 mm to (162.2, 59.1), turned to 90 degrees
- renumbered J2 to ISP, USB to J1
Connections:
- ISP pad 1: /COL0 -> /COL5
- ISP pad 3: /COL1 -> /COL4
Routing:
- net /i2c_SCL: track 46.0 -> 37.0 mm, vias 2 -> 0
- net /i2c_SDA: track 29.1 -> 31.0 mm

Commit message: Minor
Parts:
- renumbered U1 to ATmega328P, SW50 to BOOT, SW49 to RESET, J1 to USB
Other:
- outline, holes or cut-outs redrawn

Commit message: minor
Routing:
- net Net-(D48-Pad2): track 127.7 -> 124.0 mm
- net Net-(D47-Pad2): track 100.2 -> 98.2 mm
Changed lines of the file:
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@@
     (thickness 1.6)
     (drawings 28)
-    (tracks 936)
+    (tracks 934)
     (zones 0)
     (modules 124)
@@
   (segment (start 269.384018 101.479978) (end 269.38402 101.47998) (width 0.25) (layer F.Cu) (net 54))
   (segment (start 209.44716 101.479978) (end 269.384018 101.479978) (width 0.25) (layer F.Cu) (net 54))
-  (segment (start 205.187172 97.21999) (end 203.7796 97.21999) (width 0.25) (layer F.Cu) (net 54))
-  (segment (start 209.44716 101.479978) (end 205.187172 97.21999) (width 0.25) (layer F.Cu) (net 54))
-  (segment (start 203.52959 97.47) (end 201.626 97.47) (width 0.25) (layer F.Cu) (net 54))
-  (segment (start 203.7796 97.21999) (end 203.52959 97.47) (width 0.25) (layer F.Cu) (net 54))
+  (segment (start 205.43718 97.47) (end 209.44716 101.479978) (width 0.25) (layer F.Cu) (net 54))
+  (segment (start 201.626 97.47) (end 205.43718 97.47) (width 0.25) (layer F.Cu) (net 54))
   (segment (start 289.718 100.67598) (end 289.718 91.87) (width 0.25) (layer F.Cu) (net 55))
   (segment (start 288.46399 101.92999) (end 289.718 100.67598) (width 0.25) (layer F.Cu) (net 55))
-  (segment (start 201.626 100.01) (end 203.966 97.67) (width 0.25) (layer F.Cu) (net 55))
-  (segment (start 203.966 97.67) (end 205.000771 97.67) (width 0.25) (layer F.Cu) (net 55))
-  (segment (start 205.000771 97.67) (end 205.000771 97.670771) (width 0.25) (layer F.Cu) (net 55))
   (segment (start 288.463988 101.929988) (end 288.46399 101.92999) (width 0.25) (layer F.Cu) (net 55))
   (segment (start 209.259988 101.929988) (end 288.463988 101.929988) (width 0.25) (layer F.Cu) (net 55))
-  (segment (start 205.000771 97.670771) (end 209.259988 101.929988) (width 0.25) (layer F.Cu) (net 55))
+  (segment (start 202.75737 100.01) (end 202.76737 100) (width 0.25) (layer F.Cu) (net 55))
+  (segment (start 201.626 100.01) (end 202.75737 100.01) (width 0.25) (layer F.Cu) (net 55))
+  (segment (start 207.33 100) (end 209.259988 101.929988) (width 0.25) (layer F.Cu) (net 55))
+  (segment (start 202.76737 100) (end 207.33 100) (width 0.25) (layer F.Cu) (net 55))
   (segment (start 308.768 100.996) (end 308.768 91.87) (width 0.25) (layer F.Cu) (net 56))
   (segment (start 301.267002 102.38) (end 301.277002 102.39) (width 0.25) (layer F.Cu) (net 56))
   (segment (start 301.277002 102.39) (end 307.374 102.39) (width 0.25) (layer F.Cu) (net 56))
   (segment (start 307.374 102.39) (end 308.768 100.996) (width 0.25) (layer F.Cu) (net 56))
-  (segment (start 201.626 102.55) (end 203.08 101.096) (width 0.25) (layer F.Cu) (net 56))
-  (segment (start 203.08 99.2) (end 204.15999 98.12001) (width 0.25) (layer F.Cu) (net 56))
-  (segment (start 203.08 101.096) (end 203.08 99.2) (width 0.25) (layer F.Cu) (net 56))
-  (segment (start 204.15999 98.12001) (end 204.8136 98.12001) (width 0.25) (layer F.Cu) (net 56))
-  (segment (start 204.8136 98.12001) (end 209.07359 102.38) (width 0.25) (layer F.Cu) (net 56))
   (segment (start 307.364 102.38) (end 307.374 102.39) (width 0.25) (layer F.Cu) (net 56))
   (segment (start 209.07359 102.38) (end 307.364 102.38) (width 0.25) (layer F.Cu) (net 56))
+  (segment (start 209.07359 102.379998) (end 209.073587 102.379997) (width 0.25) (layer F.Cu) (net 56))
+  (segment (start 209.07359 102.38) (end 209.07359 102.379998) (width 0.25) (layer F.Cu) (net 56))
+  (segment (start 209.073587 102.379997) (end 207.94359 101.25) (width 0.25) (layer F.Cu) (net 56))
+  (segment (start 202.926 101.25) (end 201.626 102.55) (width 0.25) (layer F.Cu) (net 56))
+  (segment (start 207.94359 101.25) (end 202.926 101.25) (width 0.25) (layer F.Cu) (net 56))
   (segment (start 185.262 36.655) (end 186.312 36.655) (width 0.25) (layer F.Cu) (net 57))
   (segment (start 183.887 35.28) (end 185.262 36.655) (width 0.25) (layer F.Cu) (net 57))
@@
   (segment (start 208.3 100.42) (end 208.33999 100.38001) (width 0.25) (layer B.Cu) (net 73))
   (segment (start 176.863946 86.319) (end 175.410444 86.319) (width 0.25) (layer B.Cu) (net 73))
-  (segment (start 207.74078 100.42) (end 206.62997 99.30919) (width 0.25) (layer B.Cu) (net 73))
   (segment (start 208.3 100.42) (end 207.74078 100.42) (width 0.25) (layer B.Cu) (net 73))
   (segment (start 206.62997 99.30919) (end 206.62997 88.45997) (width 0.25) (layer B.Cu) (net 73))
@@
   (segment (start 169.250445 62.333999) (end 166.730443 62.333999) (width 0.25) (layer B.Cu) (net 73))
   (segment (start 166.27 65.41359) (end 164.60359 67.08) (width 0.25) (layer B.Cu) (net 73))
+  (segment (start 207.74078 100.42) (end 206.62997 99.30919) (width 0.25) (layer B.Cu) (net 73))
   (segment (start 315.114 33.735634) (end 315.114 51.23) (width 0.25) (layer B.Cu) (net 74))
   (segment (start 315.114 32.18) (end 315.114 33.735634) (width 0.25) (layer B.Cu) (net 74))
