File: PCB/Satellite.kicad_pcb (KiCad board)
At the start: 2 copper layers, 300 x 80 mm, 124 parts, among them SW1 SW_Push, SW10 SW_Push, SW11 SW_Push, SW12 SW_Push, SW13 SW_Push, SW14 SW_Push, SW15 SW_Push, SW16 SW_Push, SW17 SW_Push, SW18 SW_Push, SW19 SW_Push, SW2 SW_Push, SW20 SW_Push, SW21 SW_Push, SW22 SW_Push, SW23 SW_Push, SW24 SW_Push, SW25 SW_Push, SW26 SW_Push, SW27 SW_Push, SW28 SW_Push, SW29 SW_Push, SW3 SW_Push, SW30 SW_Push, SW31 SW_Push, SW32 SW_Push, SW33 SW_Push, SW34 SW_Push, SW35 SW_Push, SW36 SW_Push, SW37 SW_Push, SW38 SW_Push, SW39 SW_Push, SW4 SW_Push, SW40 SW_Push, SW41 SW_Push, SW42 SW_Push, SW43 SW_Push, SW44 SW_Push, SW45 SW_Push, SW46 SW_Push, SW47 SW_Push, SW48 SW_Push, SW5 SW_Push, SW6 SW_Push, SW7 SW_Push, SW8 SW_Push, SW9 SW_Push, Y1 16Mhz

Commit message: minor
Parts:
- removed the G*** at (185.7, 88.4)
- removed USB: USB, Custom_Footprints:USB_Mini-B_THT_Horizontal
- added J1: Conn_01x04_MountingPin, Connector_PinHeader_2.54mm:PinHeader_1x04_P2.54mm_Vertical, F.Cu at (187.1, 36.4)
- added REF**: PinHeader_1x01_P2.54mm_Vertical, Connector_PinHeader_2.54mm:PinHeader_1x01_P2.54mm_Vertical, F.Cu at (188.3, 29.1)
- moved RESET 20.9 mm to (158.7, 29.1)
- moved D50 4.12 mm to (181.2, 40.6)
- moved D49 4.11 mm to (185.3, 40.6)
- moved C3 2.00 mm to (174.5, 47.3)
- moved F1 2.00 mm to (174.4, 42.6)
- moved R3 1.34 mm to (170.3, 49.5)
- moved BOOT 1.28 mm to (168.5, 29.1)
- moved R2 0.68 mm to (165.7, 36.8)
- renumbered LED1 to GRN, LED2 to RED
Routing:
- net /COL8: track 272.3 -> 250.9 mm
- net /RESET: track 123.0 -> 107.8 mm
- net Net-(D50-Pad1): track 39.2 -> 27.7 mm
- net GND: track 173.6 -> 163.5 mm
- net Net-(F1-Pad2): track 21.2 -> 13.1 mm
- net Net-(D49-Pad1): track 26.8 -> 22.6 mm
- net +5V: track 115.9 -> 113.9 mm
Other:
- outline, holes or cut-outs redrawn

Commit message: Minor
Routing:
- added copper zone on B.Cu, net GND
- added copper zone on F.Cu, net GND
Changed lines of the file:
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@@
   (segment (start 158.21 68.38) (end 161.14 68.38) (width 0.25) (layer F.Cu) (net 62))
   (segment (start 157.779991 67.949991) (end 158.21 68.38) (width 0.25) (layer F.Cu) (net 62))
-  (segment (start 169.894213 33.64) (end 174.98 33.64) (width 0.25) (layer F.Cu) (net 75))
-  (segment (start 168.48 33.64) (end 169.894213 33.64) (width 0.25) (layer F.Cu) (net 75))
   (segment (start 175.810444 63.459) (end 175.410444 63.459) (width 0.25) (layer F.Cu) (net 63))
   (segment (start 164.21 57.4) (end 164.21 59.13) (width 0.25) (layer B.Cu) (net 63))
@@
   (segment (start 143.9236 87.85999) (end 164.08358 87.85999) (width 0.25) (layer B.Cu) (net 74))
   (segment (start 164.08358 87.85999) (end 165.54 89.31641) (width 0.25) (layer B.Cu) (net 74))
+  (segment (start 169.894213 33.64) (end 174.98 33.64) (width 0.25) (layer F.Cu) (net 75))
+  (segment (start 168.48 33.64) (end 169.894213 33.64) (width 0.25) (layer F.Cu) (net 75))
   (segment (start 75.019 33.735634) (end 75.019 51.23) (width 0.25) (layer B.Cu) (net 75))
   (segment (start 75.019 32.18) (end 75.019 33.735634) (width 0.25) (layer B.Cu) (net 75))
@@
   (segment (start 137.13 98.56995) (end 137.19995 98.56995) (width 0.25) (layer B.Cu) (net 78))
   (segment (start 141.649954 98.59995) (end 141.649957 87.587995) (width 0.25) (layer B.Cu) (net 78))
+  (zone (net 1) (net_name GND) (layer F.Cu) (hatch edge 0.508)
+    (connect_pads (clearance 0.508))
+    (min_thickness 0.254)
+    (fill yes (arc_segments 32) (thermal_gap 0.508) (thermal_bridge_width 0.508))
+    (polygon
+      (pts
+        (xy 24.86 27.74) (xy 24.86 103.93) (xy 322.1 103.93) (xy 322.1 27.73)
+      )
+    )
+  )
+  (zone (net 1) (net_name GND) (layer B.Cu) (hatch edge 0.508)
+    (connect_pads (clearance 0.508))
+    (min_thickness 0.254)
+    (fill yes (arc_segments 32) (thermal_gap 0.508) (thermal_bridge_width 0.508))
+    (polygon
+      (pts
+        (xy 24.86 27.74) (xy 24.86 103.93) (xy 322.1 103.93) (xy 322.1 27.73)
+      )
+    )
+  )
 )
