File: PCB/Satellite.kicad_pcb (KiCad board)
At the start: 2 copper layers, 300 x 80 mm, 124 parts, among them J1 Conn_01x04_MountingPin, SW1 SW_Push, SW10 SW_Push, SW11 SW_Push, SW12 SW_Push, SW13 SW_Push, SW14 SW_Push, SW15 SW_Push, SW16 SW_Push, SW17 SW_Push, SW18 SW_Push, SW19 SW_Push, SW2 SW_Push, SW20 SW_Push, SW21 SW_Push, SW22 SW_Push, SW23 SW_Push, SW24 SW_Push, SW25 SW_Push, SW26 SW_Push, SW27 SW_Push, SW28 SW_Push, SW29 SW_Push, SW3 SW_Push, SW30 SW_Push, SW31 SW_Push, SW32 SW_Push, SW33 SW_Push, SW34 SW_Push, SW35 SW_Push, SW36 SW_Push, SW37 SW_Push, SW38 SW_Push, SW39 SW_Push, SW4 SW_Push, SW40 SW_Push, SW41 SW_Push, SW42 SW_Push, SW43 SW_Push, SW44 SW_Push, SW45 SW_Push, SW46 SW_Push, SW47 SW_Push, SW48 SW_Push, SW5 SW_Push, SW6 SW_Push, SW7 SW_Push, SW8 SW_Push, SW9 SW_Push, Y1 16Mhz

Commit message: Choc_MX
Parts:
- removed the G*** at (205.2, 41.3)
- SW1, SW10, SW11, SW12, SW13, SW14, SW15, SW16, SW17, SW18, SW19, SW2, SW20, SW21, SW22, SW23, SW24, SW25, SW26, SW27, SW28, SW29, SW3, SW30, SW31, SW32, SW33, SW34, SW35, SW36, SW37, SW38, SW39, SW4, SW40, SW41, SW42, SW43, SW44, SW45, SW46, SW47, SW48, SW5, SW6, SW7, SW8, SW9: footprint MX_Alps_Hybrid:MX-1U-NoLED -> MX_Alps_Hybrid:MX_Choc_1U
Routing:
- net /COL0: track 137.1 -> 118.4 mm
- net /COL11: track 128.6 -> 112.0 mm
- net Net-(D6-Pad2): track 27.8 -> 36.2 mm
- net Net-(D5-Pad2): track 46.0 -> 53.6 mm
- net Net-(D42-Pad2): track 29.1 -> 36.2 mm
- net Net-(D30-Pad2): track 29.3 -> 36.2 mm
- net Net-(D18-Pad2): track 29.8 -> 36.2 mm
- net Net-(D4-Pad2): track 64.6 -> 70.5 mm
- net Net-(D41-Pad2): track 47.7 -> 53.6 mm
- net Net-(D29-Pad2): track 47.9 -> 53.6 mm
- net Net-(D17-Pad2): track 48.4 -> 53.6 mm
- net Net-(D3-Pad2): track 83.3 -> 87.6 mm
- net Net-(D40-Pad2): track 66.3 -> 70.5 mm
- net Net-(D28-Pad2): track 66.6 -> 70.5 mm
- net /COL10: track 146.0 -> 149.6 mm
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
Commit message: Minor update
Routing:
- net Net-(D12-Pad2): track 116.9 -> 123.8 mm
- net Net-(D24-Pad2): track 116.9 -> 123.8 mm
- net Net-(D36-Pad2): track 116.9 -> 123.8 mm
- net Net-(D32-Pad2): track 42.3 -> 46.0 mm
- net Net-(D20-Pad2): track 42.3 -> 46.0 mm
- net Net-(D8-Pad2): track 42.3 -> 46.0 mm
- net Net-(D44-Pad2): track 42.3 -> 46.0 mm
- net Net-(D9-Pad2): track 61.0 -> 63.6 mm
- net Net-(D33-Pad2): track 61.0 -> 63.6 mm
- net Net-(D21-Pad2): track 61.0 -> 63.6 mm
- net Net-(D45-Pad2): track 61.0 -> 63.6 mm
- net Net-(D34-Pad2): track 79.6 -> 80.9 mm
- net Net-(D22-Pad2): track 79.6 -> 80.9 mm
- net Net-(D10-Pad2): track 79.6 -> 80.9 mm
- net Net-(D46-Pad2): track 79.6 -> 80.9 mm
- added copper zone on B.Cu, net GND
- added copper zone on F.Cu, net GND
