File: PCB/Satellite.sch (KiCad schematic (older format))
At the start: 121 parts, among them J1 USB, J2 AVR-ISP-6, J3 I2C_Connector, SW1 SW_Push, SW10 SW_Push, SW11 SW_Push, SW12 SW_Push, SW13 SW_Push, SW14 SW_Push, SW15 SW_Push, SW16 SW_Push, SW17 SW_Push, SW18 SW_Push, SW19 SW_Push, SW2 SW_Push, SW20 SW_Push, SW21 SW_Push, SW22 SW_Push, SW23 SW_Push, SW24 SW_Push, SW25 SW_Push, SW26 SW_Push, SW27 SW_Push, SW28 SW_Push, SW29 SW_Push, SW3 SW_Push, SW30 SW_Push, SW31 SW_Push, SW32 SW_Push, SW33 SW_Push, SW34 SW_Push, SW35 SW_Push, SW36 SW_Push, SW37 SW_Push, SW38 SW_Push, SW39 SW_Push, SW4 SW_Push, SW40 SW_Push, SW41 SW_Push, SW42 SW_Push, SW43 SW_Push, SW44 SW_Push, SW45 SW_Push, SW46 SW_Push, SW47 SW_Push, SW48 SW_Push, SW49 RESET, SW5 SW_Push, SW50 BOOT, SW6 SW_Push, SW7 SW_Push, SW8 SW_Push, SW9 SW_Push, U1 ATmega328P-PU, Y1 16Mhz

Commit message: PCB minor
Connections:
- net COL0: no longer J2.1 (MISO)
- net COL1: no longer J2.3 (SCK)
- net COL4: now also J2.3 (SCK)
- net COL5: now also J2.1 (MISO)
Changed lines of the file:
@@
 EESchema Schematic File Version 4
-LIBS:vUSB_planck_keyboard-cache
 EELAYER 29 0
 EELAYER END
@@
 RESET
 Text Label 5550 4700 0    50   ~ 0
-COL1
+COL4
 Text Label 5550 4600 0    50   ~ 0
 ROW3
 Text Label 5550 4500 0    50   ~ 0
-COL0
+COL5
 Wire Wire Line
 	2450 4850 2600 4850

Commit message: minor
Parts:
- SW11: footprint Button_Switch_Keyboard:SW_Cherry_MX_1.00u_PCB -> MX_Alps_Hybrid:MX-1U-NoLED
Changed lines of the file:
@@
 F 0 "SW11" H 8800 1685 50  0000 C CNN
 F 1 "SW_Push" H 8800 1594 50  0000 C CNN
-F 2 "Button_Switch_Keyboard:SW_Cherry_MX_1.00u_PCB" H 8800 1600 50  0001 C CNN
+F 2 "MX_Alps_Hybrid:MX-1U-NoLED" H 8800 1600 50  0001 C CNN
 F 3 "~" H 8800 1600 50  0001 C CNN
 	1    8800 1400
