File: PCB/USB_Connector/USB_Connector.sch (KiCad schematic (older format))
At the start: 4 parts, among them J1 Conn_01x04_MountingPin, J2 Conn_01x04_MountingPin, J3 USB_B_Mini, P1 USB_C_Plug_USB2.0

Commit message: minor
Parts:
- added R1: 5.1k, Resistor_THT:R_Axial_DIN0309_L9.0mm_D3.2mm_P12.70mm_Horizontal, symbol Device:R
Connections:
- net GND: now reaches J1.4 (Pin_4), P1.A1 (GND), P1.A12 (GND), P1.B1 (GND), P1.B12 (GND)
- net GND: now also R1.1
- net at P1.A5 (CC): now also R1.2
Changed lines of the file:
@@
 Wire Wire Line
 	3150 3650 3150 3700
+$Comp
+L Device:R R1
+U 1 1 5CE3280B
+P 2450 950
+F 0 "R1" H 2520 996 50  0000 L CNN
+F 1 "5.1k" H 2520 905 50  0000 L CNN
+F 2 "Resistor_THT:R_Axial_DIN0309_L9.0mm_D3.2mm_P12.70mm_Horizontal" V 2380 950 50  0001 C CNN
+F 3 "~" H 2450 950 50  0001 C CNN
+	1    2450 950
+	1    0    0    -1
+$EndComp
+Wire Wire Line
+	2300 1400 2450 1400
+Wire Wire Line
+	2450 1400 2450 1100
+Wire Wire Line
+	2450 800  2450 650
+Wire Wire Line
+	2450 650  2700 650
+Text Label 2700 650  0    50   ~ 0
+GND
+Text Label 1700 2700 0    50   ~ 0
+GND
 $EndSCHEMATC
