File: PCB/USB_Connector/USB_Connector.kicad_pcb (KiCad board)
At the start: 2 copper layers, 35 x 12 mm, 8 parts, among them J1 Conn_01x04_MountingPin, J2 Conn_01x04_MountingPin

Commit message: minor
Parts:
- removed the REF** at (102.6, 29.4)
- removed the REF** at (122.6, 29.4)
- added R1: 5.1k, Resistor_SMD:R_0603_1608Metric, B.Cu at (127.9, 29.9)
- added R1: 5.1k, Resistor_SMD:R_0603_1608Metric, B.Cu at (129.9, 29.9)
- moved REF** 1.93 mm to (114.5, 31.2)
- moved REF** 1.93 mm to (134.5, 31.2)
Connections:
- net Net-(J1-Pad4) renamed /GND
- TYPE-C pad B6: (no net) -> Net-(J1-Pad2)
- TYPE-C pad B7: (no net) -> Net-(J1-Pad3)
Routing:
- net Net-(P1-PadA5): track 0.00 -> 23.4 mm, vias 0 -> 2
- net /GND: track 14.3 -> 20.1 mm
- net Net-(P1-PadB5): track 0.00 -> 5.27 mm
- net Net-(J1-Pad2): track 4.56 -> 6.24 mm
- net Net-(J1-Pad3): track 4.56 -> 6.24 mm
Other:
- board size 35 x 12 mm -> 31.2 x 12 mm

Commit message: minor
Parts:
- moved J2 8.65 mm to (113.6, 29.9), turned to 90 degrees
- moved REF** 6.58 mm to (111.8, 37.2), turned to 180 degrees
- moved MINI-B 6.43 mm to (115.8, 32.3), turned to 0 degrees
Routing:
- net Net-(J2-Pad3): track 16.5 -> 16.0 mm
Other:
- board size 31.2 x 12 mm -> 22.7 x 12 mm
